Commit message: calibration pipeline

File: src/ptu_lidar_calib/urdf/real_pantilt.urdf (robot description, URDF)
Before this commit: robot real_pantilt, 6 links, 5 joints
Links:
- link laser: geometry visual mesh filename=package://ptu_lidar_calib/urdf/meshes/URG-04LX.dae scale=0.001 0.001 0.001

Commit message: Update laser frame ID and transform checks; modify URDF mesh path and simplify HTML header

File: src/ptu_lidar_calib/urdf/real_pantilt.urdf (robot description, URDF)
Before this commit: robot real_pantilt, 6 links, 5 joints
Links:
- link laser: geometry visual mesh filename=./meshes/URG-04LX.dae scale=0.001 0.001 0.001
