Commit message: Refactor code structure for improved readability and maintainability

File: src/ptu_calib_cpp/results/calibrated_pantilt.urdf (robot description, URDF)
Before this commit: robot real_pantilt, 5 links, 4 joints
Joints:
- joint hokuyo_joint: origin xyz=-0.105860 0.016000 0.039941 rpy=-1.571469 -0.028210 1.570407 -> xyz=-0.105989 0.012000 0.040280 rpy=-1.571548 -0.033314 1.571110
- joint joint1: origin xyz=0.000027 -0.007000 0.022792 rpy=1.715387 1.535637 1.690776 -> xyz=0.000028 -0.011000 0.020879 rpy=2.321494 1.524529 2.287145
- joint joint2: origin xyz=0.000000 -0.026500 0.094000 rpy=0.034907 0.019787 -0.034907 -> xyz=0.000000 -0.030500 0.090000 rpy=0.034907 0.034907 -0.034907
