Commit message: Add comprehensive system analysis and calibration methods for PTU-LIDAR
- Introduced SYSTEM_ANALYSIS.md detailing hardware architecture, software stack, and transformation chain.
- Analyzed current calibration method, identifying limitations and proposing improvements based on IEEE paper methods.
- Implemented a two-phase calibration system in calibrate.py for data collection and offline optimization.
- Developed a script to convert calibration results to URDF format for integration into robotic systems.
- Added calibration data storage in calibration_data.npz for efficient data handling.

File: src/hokuyo_go/urdf/real_pantilt.urdf (robot description, URDF)
Before this commit: robot real_pantilt, 6 links, 5 joints
Joints:
- joint hokuyo_joint: origin xyz=-0.061 0.0140 0.033 rpy=1.57 3.14 -1.57 -> xyz=-0.061 0.0140 0.040 rpy=1.57 3.14 -1.57
- joint joint1: origin xyz=0 0 0.022 rpy=0 1.57 0 -> xyz=0 -0.009 0.022 rpy=0 1.57 0

File: src/ptu_lidar_calib/urdf/real_pantilt.urdf (robot description, URDF)
Before this commit: robot real_pantilt, 6 links, 5 joints
Links:
- link laser: geometry visual mesh filename=package://hokuyo_go/urdf/meshes/URG-04LX.dae scale=0.001 0.001 0.001
Joints:
- joint hokuyo_joint: origin xyz=-0.061 0.0140 0.033 rpy=1.57 3.14 -1.57 -> xyz=-0.061 0.0140 0.040 rpy=1.57 3.14 -1.57
- joint joint1: origin xyz=0 0 0.022 rpy=0 1.57 0 -> xyz=0 -0.009 0.022 rpy=0 1.57 0

Commit message: Add simulation joint controller and URDF models for calibration testing
- Implemented `sim_joint_controller.cpp` to bridge the real robot's interface with Gazebo joint effort commands using a PD controller for pan and tilt joints.
- Created `nominal_pantilt.urdf` representing the ground truth model of the pan-tilt mechanism.
- Developed `skewed_pantilt.urdf` for calibration testing, incorporating intentional perturbations in joint positions and orientations.
- Added `calib_test.world`, a simple Gazebo world with a flat wall for calibration testing, ensuring the laser scan plane is appropriately positioned.

File: src/hokuyo_go/urdf/real_pantilt.urdf (robot description, URDF)
Before this commit: robot real_pantilt, 5 links, 4 joints
Links:
- added link hokuyo_base, mass 0.10; visual box size=0.162 0.06 0.003
Joints:
- added joint hokuyo_base_joint: type fixed, parent tilt_link, child hokuyo_base, origin xyz=-0.0450 0 0 rpy=0 0 0
- joint hokuyo_joint: origin xyz=-0.105860 0.016000 0.039941 rpy=-1.571469 -0.028210 1.570407 -> xyz=-0.061 0.0140 0.040 rpy=1.57 3.14 -1.57; parent tilt_link -> hokuyo_base
- joint joint1: origin xyz=0.000027 -0.007000 0.022792 rpy=1.715387 1.535637 1.690776 -> xyz=0 -0.009 0.022 rpy=0 1.57 0
- joint joint2: origin xyz=0.000000 -0.026500 0.094000 rpy=0.034907 0.019787 -0.034907 -> xyz=0 -0.0285 0.092 rpy=0 0 0

File: src/ptu_calib_cpp/results/calibrated_pantilt.urdf (robot description, URDF)
Before this commit: robot real_pantilt, 5 links, 4 joints
Joints:
- joint hokuyo_joint: origin xyz=-0.105989 0.012000 0.040280 rpy=-1.571548 -0.033314 1.571110 -> xyz=-0.106000 0.014000 0.040000 rpy=-1.571593 0.001593 1.571593
- joint joint1: origin xyz=0.000028 -0.011000 0.020879 rpy=2.321494 1.524529 2.287145 -> xyz=-0.000001 -0.006070 0.022373 rpy=1.693000 1.518278 1.648727
- joint joint2: origin xyz=0.000000 -0.030500 0.090000 rpy=0.034907 0.034907 -0.034907 -> xyz=0.000000 -0.025500 0.095000 rpy=0.052360 0.000860 -0.001166
